Commit message: rename xarm to xarm7

File: xarm7_description/urdf/gripper/gripper.urdf.xacro (robot description, xacro)
@@ -4,5 +4,5 @@
   <xacro:arg name="prefix" default=""/>
   <xacro:arg name="mesh_suffix" default="stl"/>
-  <xacro:include filename="$(find xarm_description)/urdf/gripper/gripper_macro.xacro" />
+  <xacro:include filename="$(find xarm7_description)/urdf/gripper/gripper_macro.xacro" />
   <xacro:gripper_device robot_type="$(arg robot_type)" prefix="$(arg prefix)" mesh_suffix="$(arg mesh_suffix)" />
 </robot>

File: xarm7_description/urdf/gripper/gripper_macro.xacro (robot description, xacro)
@@ -3,25 +3,25 @@
   <xacro:macro name="gripper_device" params="prefix:='' robot_type:='xarm' mesh_suffix:='stl' ">
     <!-- Load Common Material -->
-    <xacro:include filename="$(find xarm_description)/urdf/_private_macro.xacro" />
+    <xacro:include filename="$(find xarm7_description)/urdf/_private_macro.xacro" />
     <xacro:device_macro_begin />
     <!-- Load Common Material -->
-    <xacro:include filename="$(find xarm_description)/urdf/common/common.material.xacro" />
+    <xacro:include filename="$(find xarm7_description)/urdf/common/common.material.xacro" />
     <xacro:common_material prefix="${prefix}"/>
-    <xacro:property name="mesh_path" value="package://xarm_description/meshes" scope="parent"/>
+    <xacro:property name="mesh_path" value="package://xarm7_description/meshes" scope="parent"/>
     <!-- include common.link.xacro -->
-    <xacro:include filename="$(find xarm_description)/urdf/common/common.link.xacro" />
+    <xacro:include filename="$(find xarm7_description)/urdf/common/common.link.xacro" />
     <xacro:if value="${robot_type == 'lite'}">
       <!-- Load Lite Gripper Model URDF -->
-      <xacro:include filename="$(find xarm_description)/urdf/gripper/lite_gripper.urdf.xacro" />
+      <xacro:include filename="$(find xarm7_description)/urdf/gripper/lite_gripper.urdf.xacro" />
       <xacro:uflite_gripper_urdf prefix="${prefix}" />
     </xacro:if>
     <xacro:if value="${robot_type == 'bio'}">
       <!-- Load BIO Gripper Model URDF -->
-      <xacro:include filename="$(find xarm_description)/urdf/gripper/bio_gripper_macro.xacro" />
+      <xacro:include filename="$(find xarm7_description)/urdf/gripper/bio_gripper_macro.xacro" />
       <xacro:bio_gripper_macro prefix="${prefix}" />
     </xacro:if>
     <xacro:unless value="${robot_type == 'lite' or robot_type == 'bio'}">
       <!-- Load XArm Gripper Model URDF -->
-      <xacro:include filename="$(find xarm_description)/urdf/gripper/xarm_gripper_macro.xacro" />
+      <xacro:include filename="$(find xarm7_description)/urdf/gripper/xarm_gripper_macro.xacro" />
       <xacro:xarm_gripper_macro prefix="${prefix}" />
     </xacro:unless>

File: xarm7_description/urdf/gripper/xarm_gripper_macro.xacro (robot description, xacro)
@@ -2,8 +2,8 @@
 <robot xmlns:xacro="http://ros.org/wiki/xacro" name="xarm_gripper" >
   <!-- xarm_gripper -->
-  <xacro:include filename="$(find xarm_description)/urdf/gripper/xarm_gripper.ros2_control.xacro" />
-  <xacro:include filename="$(find xarm_description)/urdf/gripper/xarm_gripper.urdf.xacro" />
-  <xacro:include filename="$(find xarm_description)/urdf/gripper/xarm_gripper.transmission.xacro" />
-  <xacro:include filename="$(find xarm_description)/urdf/gripper/xarm_gripper.gazebo.xacro" />
+  <xacro:include filename="$(find xarm7_description)/urdf/gripper/xarm_gripper.ros2_control.xacro" />
+  <xacro:include filename="$(find xarm7_description)/urdf/gripper/xarm_gripper.urdf.xacro" />
+  <xacro:include filename="$(find xarm7_description)/urdf/gripper/xarm_gripper.transmission.xacro" />
+  <xacro:include filename="$(find xarm7_description)/urdf/gripper/xarm_gripper.gazebo.xacro" />
   <xacro:macro name="xarm_gripper_macro" params="prefix:='' attach_to:='' ns:='xarm' attach_xyz:='0 0 0' attach_rpy:='0 0 0'
     ros2_control_plugin:='uf_robot_hardware/UFRobotFakeSystemHardware' dof:=7 hard_interface:='PositionJointInterface' ">

File: xarm7_description/urdf/xarm7/xarm7.urdf.xacro (robot description, xacro)
@@ -38,8 +38,8 @@
     <xacro:property name="default_inertial_params_filename" value="xarm7_type7_HT_BR2"/>
     <xacro:if value="${inertial_params_filename != ''}">
-      <xacro:property name="link_inertial_params_file" value="$(find xarm_description)/config/link_inertial/${inertial_params_filename}.yaml"/>
+      <xacro:property name="link_inertial_params_file" value="$(find xarm7_description)/config/link_inertial/${inertial_params_filename}.yaml"/>
     </xacro:if>
     <xacro:unless value="${inertial_params_filename != ''}">
-      <xacro:property name="link_inertial_params_file" value="$(find xarm_description)/config/link_inertial/${default_inertial_params_filename}.yaml"/>
+      <xacro:property name="link_inertial_params_file" value="$(find xarm7_description)/config/link_inertial/${default_inertial_params_filename}.yaml"/>
     </xacro:unless>
     <xacro:if value="${use_xacro_load_yaml}">

File: xarm7_description/urdf/xarm7/xarm7_robot_macro.xacro (robot description, xacro)
@@ -20,9 +20,9 @@
     <!-- xarm7 -->
     <xacro:if value="${is_ros2}">
-      <xacro:include filename="$(find xarm_description)/urdf/xarm7/xarm7.ros2_control.xacro" />
+      <xacro:include filename="$(find xarm7_description)/urdf/xarm7/xarm7.ros2_control.xacro" />
     </xacro:if>
-    <xacro:include filename="$(find xarm_description)/urdf/xarm7/xarm7.urdf.xacro" />
-    <xacro:include filename="$(find xarm_description)/urdf/xarm7/xarm7.transmission.xacro" />
-    <xacro:include filename="$(find xarm_description)/urdf/xarm7/xarm7.gazebo.xacro" />
+    <xacro:include filename="$(find xarm7_description)/urdf/xarm7/xarm7.urdf.xacro" />
+    <xacro:include filename="$(find xarm7_description)/urdf/xarm7/xarm7.transmission.xacro" />
+    <xacro:include filename="$(find xarm7_description)/urdf/xarm7/xarm7.gazebo.xacro" />
     <xacro:if value="${limited}">
       <xacro:if value="${is_ros2}">

File: xarm7_description/urdf/xarm_device.urdf.xacro (robot description, xacro)
@@ -40,5 +40,5 @@
   <xacro:arg name="kinematics_suffix" default=""/>
   <!-- load xarm device -->
-  <xacro:include filename="$(find xarm_description)/urdf/xarm_device_macro.xacro" />
+  <xacro:include filename="$(find xarm7_description)/urdf/xarm_device_macro.xacro" />
   <xacro:xarm_device prefix="$(arg prefix)" hw_ns="$(arg hw_ns)" limited="$(arg limited)"
     effort_control="$(arg effort_control)" velocity_control="$(arg velocity_control)"

File: xarm7_description/urdf/xarm_device_macro.xacro (robot description, xacro)
@@ -45,8 +45,8 @@
     >
     <!-- Load Common Material -->
-    <xacro:include filename="$(find xarm_description)/urdf/_private_macro.xacro" />
+    <xacro:include filename="$(find xarm7_description)/urdf/_private_macro.xacro" />
     <xacro:device_macro_begin />
     <!-- Load Common Material -->
-    <xacro:include filename="$(find xarm_description)/urdf/common/common.material.xacro" />
+    <xacro:include filename="$(find xarm7_description)/urdf/common/common.material.xacro" />
     <xacro:common_material prefix="${prefix}"/>
     <!-- Specify Mesh file path -->
@@ -54,11 +54,11 @@
     <xacro:if value="${ros2_control_plugin == 'gazebo_ros2_control/GazeboSystem' or ros2_control_plugin == 'ign_ros2_control/IgnitionSystem'}">
       <!-- gazebo use -->
-      <xacro:property name="mesh_path" value="file://$(find xarm_description)/meshes" scope="parent"/>
+      <xacro:property name="mesh_path" value="file://$(find xarm7_description)/meshes" scope="parent"/>
     </xacro:if>
     <xacro:unless value="${ros2_control_plugin == 'gazebo_ros2_control/GazeboSystem' or ros2_control_plugin == 'ign_ros2_control/IgnitionSystem'}">
-      <xacro:property name="mesh_path" value="package://xarm_description/meshes" scope="parent"/>
+      <xacro:property name="mesh_path" value="package://xarm7_description/meshes" scope="parent"/>
     </xacro:unless>
     <!-- include common.link.xacro -->
-    <xacro:include filename="$(find xarm_description)/urdf/common/common.link.xacro" />
+    <xacro:include filename="$(find xarm7_description)/urdf/common/common.link.xacro" />
     <xacro:parse_link_inertial_filename dof="${dof}" robot_type="${robot_type}" robot_sn="${robot_sn}" model1300="${model1300}" />
     <xacro:property name="inertial_params_filename" value="${scope_parent_inertial_params_filename}"/>
@@ -91,12 +91,12 @@
     </xacro:unless>
     <xacro:if value="${kinematics_suffix != ''}">
-      <xacro:property name="kinematics_params_filename" value="$(find xarm_description)/config/kinematics/user/${robot_name}_kinematics_${kinematics_suffix}.yaml"/>
+      <xacro:property name="kinematics_params_filename" value="$(find xarm7_description)/config/kinematics/user/${robot_name}_kinematics_${kinematics_suffix}.yaml"/>
     </xacro:if>
     <xacro:unless value="${kinematics_suffix != ''}">
-      <xacro:property name="kinematics_params_filename" value="$(find xarm_description)/config/kinematics/default/${robot_name}_default_kinematics.yaml"/>
+      <xacro:property name="kinematics_params_filename" value="$(find xarm7_description)/config/kinematics/default/${robot_name}_default_kinematics.yaml"/>
     </xacro:unless>
     <xacro:if value="${dof == 5}">
       <!-- Load XArm5 Robot Model URDF -->
-      <xacro:include filename="$(find xarm_description)/urdf/xarm5/xarm5_robot_macro.xacro" />
+      <xacro:include filename="$(find xarm7_description)/urdf/xarm5/xarm5_robot_macro.xacro" />
       <xacro:xarm5_robot prefix="${prefix}" hw_ns="${hw_ns}" limited="${limited}"
         velocity_control="${velocity_control}"
@@ -116,5 +116,5 @@
       <xacro:if value="${robot_type == 'uf850'}">
         <!-- Load UFACTORY 850 Robot Model URDF -->
-        <xacro:include filename="$(find xarm_description)/urdf/uf850/uf850_robot_macro.xacro" />
+        <xacro:include filename="$(find xarm7_description)/urdf/uf850/uf850_robot_macro.xacro" />
         <xacro:uf850_robot prefix="${prefix}" hw_ns="${hw_ns}" limited="${limited}"
           velocity_control="${velocity_control}"
@@ -133,5 +133,5 @@
       <xacro:if value="${robot_type == 'lite'}">
         <!-- Load Lite6 Robot Model URDF -->
-        <xacro:include filename="$(find xarm_description)/urdf/lite6/lite6_robot_macro.xacro" />
+        <xacro:include filename="$(find xarm7_description)/urdf/lite6/lite6_robot_macro.xacro" />
         <xacro:lite6_robot prefix="${prefix}" hw_ns="${hw_ns}" limited="${limited}"
           velocity_control="${velocity_control}"
@@ -149,5 +149,5 @@
       <xacro:unless value="${robot_type == 'lite' or robot_type == 'uf850'}">
         <!-- Load XArm6 Robot Model URDF -->
-        <xacro:include filename="$(find xarm_description)/urdf/xarm6/xarm6_robot_macro.xacro" />
+        <xacro:include filename="$(find xarm7_description)/urdf/xarm6/xarm6_robot_macro.xacro" />
         <xacro:xarm6_robot prefix="${prefix}" hw_ns="${hw_ns}" limited="${limited}"
           velocity_control="${velocity_control}"
@@ -168,5 +168,5 @@
       <xacro:if value="${robot_type == 'xarm7_mirror'}">
         <!-- Load xArm7 Mirror Robot Model URDF -->
-        <xacro:include filename="$(find xarm_description)/urdf/xarm7_mirror/xarm7_mirror_robot_macro.xacro" />
+        <xacro:include filename="$(find xarm7_description)/urdf/xarm7_mirror/xarm7_mirror_robot_macro.xacro" />
         <xacro:xarm7_mirror_robot prefix="${prefix}" hw_ns="${hw_ns}" limited="${limited}"
           velocity_control="${velocity_control}"
@@ -185,5 +185,5 @@
       <xacro:unless value="${robot_type == 'xarm7_mirror'}">
         <!-- Load XArm7 Robot Model URDF -->
-        <xacro:include filename="$(find xarm_description)/urdf/xarm7/xarm7_robot_macro.xacro" />
+        <xacro:include filename="$(find xarm7_description)/urdf/xarm7/xarm7_robot_macro.xacro" />
         <xacro:xarm7_robot prefix="${prefix}" hw_ns="${hw_ns}" limited="${limited}"
           velocity_control="${velocity_control}"
@@ -203,8 +203,8 @@
     <xacro:if value="${add_realsense_d435i}">
       <!-- (xarm) Load RealSense D435i URDF -->
-      <xacro:include filename="$(find xarm_description)/urdf/camera/realsense_d435i.urdf.xacro" />
+      <xacro:include filename="$(find xarm7_description)/urdf/camera/realsense_d435i.urdf.xacro" />
       <xacro:d435i_urdf prefix="${prefix}" add_d435i_links="${add_d435i_links}" />
       <xacro:if value="${add_d435i_links}">
-        <xacro:include filename="$(find xarm_description)/urdf/camera/realsense.gazebo.xacro" />
+        <xacro:include filename="$(find xarm7_description)/urdf/camera/realsense.gazebo.xacro" />
         <xacro:realsense_gazebo prefix="${prefix}" />
       </xacro:if>
@@ -221,10 +221,10 @@
       <xacro:if value="${robot_type == 'lite'}">
         <!-- Load Lite Gripper Model URDF -->
-        <xacro:include filename="$(find xarm_description)/urdf/gripper/lite_gripper.urdf.xacro" />
+        <xacro:include filename="$(find xarm7_description)/urdf/gripper/lite_gripper.urdf.xacro" />
         <xacro:uflite_gripper_urdf prefix="${prefix}" attach_to="${prefix}link_eef" />
       </xacro:if>
       <xacro:unless value="${robot_type == 'lite'}">
         <!-- Load XArm Gripper Model URDF -->
-        <xacro:include filename="$(find xarm_description)/urdf/gripper/xarm_gripper_macro.xacro" />
+        <xacro:include filename="$(find xarm7_description)/urdf/gripper/xarm_gripper_macro.xacro" />
         <xacro:xarm_gripper_macro prefix="${prefix}" attach_to="${prefix}link_eef"
           ros2_control_plugin="${ros2_control_plugin}" dof="${dof}" hard_interface="${hard_interface}" />
@@ -234,5 +234,5 @@
       <xacro:unless value="${robot_type == 'lite'}">
         <!-- Load BIO Gripper Model URDF -->
-        <xacro:include filename="$(find xarm_description)/urdf/gripper/bio_gripper_macro.xacro" />
+        <xacro:include filename="$(find xarm7_description)/urdf/gripper/bio_gripper_macro.xacro" />
         <xacro:bio_gripper_macro prefix="${prefix}" attach_to="${prefix}link_eef"
           ros2_control_plugin="${ros2_control_plugin}" dof="${dof}" hard_interface="${hard_interface}" />
@@ -242,10 +242,10 @@
       <xacro:if value="${robot_type == 'lite'}">
         <!-- Load Lite Vacuum Gripper Model URDF -->
-        <xacro:include filename="$(find xarm_description)/urdf/vacuum_gripper/lite_vacuum_gripper.urdf.xacro" />
+        <xacro:include filename="$(find xarm7_description)/urdf/vacuum_gripper/lite_vacuum_gripper.urdf.xacro" />
         <xacro:uflite_vacuum_gripper_urdf prefix="${prefix}" attach_to="${prefix}link_eef" />
       </xacro:if>
       <xacro:unless value="${robot_type == 'lite'}">
         <!-- Load XArm Vacuum Gripper Model URDF -->
-        <xacro:include filename="$(find xarm_description)/urdf/vacuum_gripper/xarm_vacuum_gripper.urdf.xacro" />
+        <xacro:include filename="$(find xarm7_description)/urdf/vacuum_gripper/xarm_vacuum_gripper.urdf.xacro" />
         <xacro:xarm_vacuum_gripper_urdf prefix="${prefix}" attach_to="${prefix}link_eef" />
       </xacro:unless>
@@ -253,5 +253,5 @@
     <xacro:if value="${not add_gripper and not add_vacuum_gripper and add_other_geometry}">
       <!-- Load Other Model URDF -->
-      <xacro:include filename="$(find xarm_description)/urdf/other/other_geometry.urdf.xacro" />
+      <xacro:include filename="$(find xarm7_description)/urdf/other/other_geometry.urdf.xacro" />
       <xacro:other_geometry prefix="${prefix}" attach_to="${prefix}link_eef"
         geometry_type="${geometry_type}" geometry_mass="${geometry_mass}"
@@ -265,5 +265,5 @@
     <!-- gazebo_plugin -->
     <xacro:if value="${load_gazebo_plugin}">
-      <xacro:include filename="$(find xarm_description)/urdf/common/common.gazebo.xacro" />
+      <xacro:include filename="$(find xarm7_description)/urdf/common/common.gazebo.xacro" />
       <xacro:if value="${is_ros2}">
         <xacro:if value="${robot_type == 'uf850' or robot_type == 'xarm7_mirror'}">
@@ -291,5 +291,5 @@
     </xacro:if>
     <xacro:if value="${use_gazebo_camera}">
-      <xacro:include filename="$(find xarm_description)/urdf/camera/camera.gazebo.xacro" />
+      <xacro:include filename="$(find xarm7_description)/urdf/camera/camera.gazebo.xacro" />
       <xacro:camera_gazebo prefix="${prefix}" />
     </xacro:if>

File: xarm7_moveit_config/srdf/xarm.srdf.xacro (robot description, xacro)
@@ -9,5 +9,5 @@
   <xacro:arg name="add_bio_gripper" default="false" />
   <xacro:arg name="add_other_geometry" default="false" />
-  <xacro:include filename="$(find xarm_moveit_config)/srdf/xarm_macro.srdf.xacro" />
+  <xacro:include filename="$(find xarm7_moveit_config)/srdf/xarm_macro.srdf.xacro" />
   <xacro:xarm_macro_srdf prefix="$(arg prefix)" dof="$(arg dof)" robot_type="$(arg robot_type)"
     add_gripper="$(arg add_gripper)" add_vacuum_gripper="$(arg add_vacuum_gripper)" add_bio_gripper="$(arg add_bio_gripper)" add_other_geometry="$(arg add_other_geometry)" />

File: xarm7_moveit_config/srdf/xarm_macro.srdf.xacro (robot description, xacro)
@@ -4,5 +4,5 @@
     add_gripper:='false' add_vacuum_gripper:='false' add_bio_gripper:='false' add_other_geometry:='false' ">
     <xacro:if value="${dof == 5}">
-      <xacro:include filename="$(find xarm_moveit_config)/srdf/_xarm5_macro.srdf.xacro" />
+      <xacro:include filename="$(find xarm7_moveit_config)/srdf/_xarm5_macro.srdf.xacro" />
       <xacro:xarm5_macro_srdf prefix="${prefix}"
         add_gripper="${add_gripper}" add_vacuum_gripper="${add_vacuum_gripper}" add_bio_gripper="${add_bio_gripper}" add_other_geometry="${add_other_geometry}" />
@@ -10,15 +10,15 @@
     <xacro:if value="${dof == 6}">
       <xacro:if value="${robot_type == 'uf850'}">
-        <xacro:include filename="$(find xarm_moveit_config)/srdf/_uf850_macro.srdf.xacro" />
+        <xacro:include filename="$(find xarm7_moveit_config)/srdf/_uf850_macro.srdf.xacro" />
         <xacro:uf850_macro_srdf prefix="${prefix}"
           add_gripper="${add_gripper}" add_vacuum_gripper="${add_vacuum_gripper}" add_bio_gripper="${add_bio_gripper}" add_other_geometry="${add_other_geometry}"  />
       </xacro:if>
       <xacro:if value="${robot_type == 'lite'}">
-        <xacro:include filename="$(find xarm_moveit_config)/srdf/_lite6_macro.srdf.xacro" />
+        <xacro:include filename="$(find xarm7_moveit_config)/srdf/_lite6_macro.srdf.xacro" />
         <xacro:lite6_macro_srdf prefix="${prefix}"
           add_gripper="${add_gripper}" add_vacuum_gripper="${add_vacuum_gripper}" add_other_geometry="${add_other_geometry}"  />
       </xacro:if>
       <xacro:unless value="${robot_type == 'lite' or robot_type == 'uf850'}">
-        <xacro:include filename="$(find xarm_moveit_config)/srdf/_xarm6_macro.srdf.xacro" />
+        <xacro:include filename="$(find xarm7_moveit_config)/srdf/_xarm6_macro.srdf.xacro" />
         <xacro:xarm6_macro_srdf prefix="${prefix}"
           add_gripper="${add_gripper}" add_vacuum_gripper="${add_vacuum_gripper}" add_bio_gripper="${add_bio_gripper}" add_other_geometry="${add_other_geometry}"  />
@@ -27,10 +27,10 @@
     <xacro:unless value="${dof == 5 or dof == 6}">
       <xacro:if value="${robot_type == 'xarm7_mirror'}">
-        <xacro:include filename="$(find xarm_moveit_config)/srdf/_xarm7_mirror_macro.srdf.xacro" />
+        <xacro:include filename="$(find xarm7_moveit_config)/srdf/_xarm7_mirror_macro.srdf.xacro" />
         <xacro:xarm7_mirror_macro_srdf prefix="${prefix}"
           add_gripper="${add_gripper}" add_vacuum_gripper="${add_vacuum_gripper}" add_bio_gripper="${add_bio_gripper}" add_other_geometry="${add_other_geometry}"  />
       </xacro:if>
       <xacro:unless value="${robot_type == 'xarm7_mirror'}">
-        <xacro:include filename="$(find xarm_moveit_config)/srdf/_xarm7_macro.srdf.xacro" />
+        <xacro:include filename="$(find xarm7_moveit_config)/srdf/_xarm7_macro.srdf.xacro" />
         <xacro:xarm7_macro_srdf prefix="${prefix}"
           add_gripper="${add_gripper}" add_vacuum_gripper="${add_vacuum_gripper}" add_bio_gripper="${add_bio_gripper}" add_other_geometry="${add_other_geometry}"  />
